Commit message: demo using kuka dynamics

File: robot_models/kuka_iiwa/kuka_iiwa.urdf (robot description, URDF)
Before this commit: robot kuka_iiwa, 8 links, 7 joints
Links:
- link link6: geometry visual mesh filename=meshes/link6.obj scale=1 1 1

Commit message: final cs225A demo

File: robot_models/kuka_iiwa/kuka_iiwa.urdf (robot description, URDF)
Before this commit: robot kuka_iiwa, 8 links, 7 joints
Joints:
- joint j3: axis 0 1 0 -> 0 -1 0
