Commit message: changed build structure so different applications have subfolders in bin

File: robot_models/kuka_iiwa/01-force_tracking/kuka_iiwa.urdf (robot description, URDF)
Before this commit: robot kuka_iiwa, 9 links, 8 joints
Links:
- removed link end_effector
- link base_link: geometry visual mesh filename=../meshes/base.obj scale=1 1 1
- link link0: geometry visual mesh filename=../meshes/link0.obj scale=1 1 1
- link link1: geometry visual mesh filename=../meshes/link1.obj scale=1 1 1
- link link2: geometry visual mesh filename=../meshes/link2.obj scale=1 1 1
- link link3: geometry visual mesh filename=../meshes/link3.obj scale=1 1 1
- link link4: geometry visual mesh filename=../meshes/link4.obj scale=1 1 1
- link link5: geometry visual mesh filename=../meshes/link5.obj scale=1 1 1
- link link6: geometry collision mesh filename=../meshes/link6.obj scale=1 1 1; visual mesh filename=../meshes/link6.obj scale=1 1 1
Joints:
- removed joint force_sensor
- joint j0: origin xyz=0.000000 0.000000 0.155767 rpy=-0.000000 0.000000 -0.000000 -> xyz=0.000000 0.000000 0.155767 rpy=0.000000 0.000000 0.000000
- joint j1: origin xyz=0.000000 0.000000 0.182500 rpy=-0.000000 0.000000 -0.000000 -> xyz=0.000000 0.000000 0.182500 rpy=0.000000 0.000000 0.000000
- joint j2: origin xyz=0.000000 0.000000 0.185000 rpy=-0.000000 0.000000 -0.000000 -> xyz=0.000000 0.000000 0.185000 rpy=0.000000 0.000000 0.000000
- joint j5: origin xyz=0.000000 0.000000 0.217003 rpy=-0.000000 0.000000 -0.000000 -> xyz=0.000000 0.000000 0.217003 rpy=0.000000 0.000000 0.000000
- joint j6: origin xyz=0.000000 0.000000 0.081000 rpy=-0.000000 0.000000 -0.000000 -> xyz=0.000000 0.000000 0.081000 rpy=0.000000 0.000000 0.000000

File: robot_models/kuka_iiwa/01-force_tracking/kuka_iiwa_force_sensor.urdf (robot description, URDF)
Before this commit: robot kuka_iiwa, 9 links, 8 joints
Links:
- link base_link: geometry visual mesh filename=../meshes/base.obj scale=1 1 1
- link link0: geometry visual mesh filename=../meshes/link0.obj scale=1 1 1
- link link1: geometry visual mesh filename=../meshes/link1.obj scale=1 1 1
- link link2: geometry visual mesh filename=../meshes/link2.obj scale=1 1 1
- link link3: geometry visual mesh filename=../meshes/link3.obj scale=1 1 1
- link link4: geometry visual mesh filename=../meshes/link4.obj scale=1 1 1
- link link5: geometry visual mesh filename=../meshes/link5.obj scale=1 1 1
- link link6: geometry collision mesh filename=../meshes/link6.obj scale=1 1 1; visual mesh filename=../meshes/link6.obj scale=1 1 1
Joints:
- joint j0: origin xyz=0.000000 0.000000 0.155767 rpy=-0.000000 0.000000 -0.000000 -> xyz=0.000000 0.000000 0.155767 rpy=0.000000 0.000000 0.000000
- joint j1: origin xyz=0.000000 0.000000 0.182500 rpy=-0.000000 0.000000 -0.000000 -> xyz=0.000000 0.000000 0.182500 rpy=0.000000 0.000000 0.000000
- joint j2: origin xyz=0.000000 0.000000 0.185000 rpy=-0.000000 0.000000 -0.000000 -> xyz=0.000000 0.000000 0.185000 rpy=0.000000 0.000000 0.000000
- joint j5: origin xyz=0.000000 0.000000 0.217003 rpy=-0.000000 0.000000 -0.000000 -> xyz=0.000000 0.000000 0.217003 rpy=0.000000 0.000000 0.000000
- joint j6: origin xyz=0.000000 0.000000 0.081000 rpy=-0.000000 0.000000 -0.000000 -> xyz=0.000000 0.000000 0.081000 rpy=0.000000 0.000000 0.000000

File: robot_models/kuka_iiwa/kuka_iiwa.urdf (robot description, URDF)
Before this commit: robot kuka_iiwa, 8 links, 7 joints
Links:
- link base_link: geometry visual mesh filename=kuka_iiwa_graphics/base.obj scale=1 1 1
- link link0: geometry visual mesh filename=kuka_iiwa_graphics/link0.obj scale=1 1 1
- link link1: geometry visual mesh filename=kuka_iiwa_graphics/link1.obj scale=1 1 1
- link link2: geometry visual mesh filename=kuka_iiwa_graphics/link2.obj scale=1 1 1
- link link3: geometry visual mesh filename=kuka_iiwa_graphics/link3.obj scale=1 1 1
- link link4: geometry visual mesh filename=kuka_iiwa_graphics/link4.obj scale=1 1 1
- link link5: geometry visual mesh filename=kuka_iiwa_graphics/link5.obj scale=1 1 1
- link link6: geometry collision mesh filename=kuka_iiwa_graphics/link6.obj scale=1 1 1; visual mesh filename=kuka_iiwa_graphics/link6.obj scale=1 1 1
Joints:
- joint j0: origin xyz=0.000000 0.000000 0.155767 rpy=-0.000000 0.000000 -0.000000 -> xyz=0.000000 0.000000 0.155767 rpy=0.000000 0.000000 0.000000
- joint j1: origin xyz=0.000000 0.000000 0.182500 rpy=-0.000000 0.000000 -0.000000 -> xyz=0.000000 0.000000 0.182500 rpy=0.000000 0.000000 0.000000
- joint j2: origin xyz=0.000000 0.000000 0.185000 rpy=-0.000000 0.000000 -0.000000 -> xyz=0.000000 0.000000 0.185000 rpy=0.000000 0.000000 0.000000
- joint j3: axis 0 -1 0 -> 0 1 0; origin xyz=0.000000 0.000000 0.217000 rpy=-0.000000 0.000000 -0.000000 -> xyz=0.000000 0.000000 0.217000 rpy=0.000000 0.000000 3.1415926535897
- joint j4: origin xyz=0.000000 0.000000 0.186000 rpy=-0.000000 0.000000 -0.000000 -> xyz=0.000000 0.000000 0.186000 rpy=0.000000 0.000000 -3.1415926535897
- joint j5: origin xyz=0.000000 0.000000 0.217003 rpy=-0.000000 0.000000 -0.000000 -> xyz=0.000000 0.000000 0.217003 rpy=0.000000 0.000000 0.000000
- joint j6: origin xyz=0.000000 0.000000 0.081000 rpy=-0.000000 0.000000 -0.000000 -> xyz=0.000000 0.000000 0.081000 rpy=0.000000 0.000000 0.000000
