Commit message: added application with 3DOF force sensor at the base and end effector

File: robot_models/kuka_iiwa/03-multi_contact_validation/kuka_iiwa_base_sensor.urdf (robot description, URDF)
Before this commit: robot kuka_iiwa, 8 links, 7 joints
Links:
- added link dummy_base_sensor_link0, mass 0.001
- added link dummy_base_sensor_link1, mass 0.001
- added link dummy_base_sensor_link2, mass 0.001
- added link dummy_ee_sensor_link0, mass 0.001
- added link dummy_ee_sensor_link1, mass 0.001
- added link end_effector, mass 0.5; collision sphere radius=0.035; visual sphere radius=0.035
- link link6: geometry visual mesh filename=../meshes/link6.obj scale=1 1 1
Joints:
- added joint fsbase_x: type prismatic, parent dummy_base_sensor_link0, child dummy_base_sensor_link1, origin xyz=0.000000 0.000000 0.00000 rpy=0.000000 0.000000 0.000000, axis 1 0 0, limit lower=-0.001 upper=0.001 effort=400 velocity=100
- added joint fsbase_y: type prismatic, parent dummy_base_sensor_link1, child dummy_base_sensor_link2, origin xyz=0.000000 0.000000 0.00000 rpy=0.000000 0.000000 0.000000, axis 0 1 0, limit lower=-0.001 upper=0.001 effort=400 velocity=100
- added joint fsbase_z: type prismatic, parent dummy_base_sensor_link2, child base_link, origin xyz=0.000000 0.000000 0.00000 rpy=0.000000 0.000000 0.000000, axis 0 0 1, limit lower=-0.001 upper=0.001 effort=400 velocity=100
- added joint fsee_x: type prismatic, parent link6, child dummy_ee_sensor_link0, origin xyz=0.000000 0.000000 0.00000 rpy=0.000000 0.000000 0.000000, axis 1 0 0, limit lower=-0.001 upper=0.001 effort=400 velocity=100
- added joint fsee_y: type prismatic, parent dummy_ee_sensor_link0, child dummy_ee_sensor_link1, origin xyz=0.000000 0.000000 0.00000 rpy=0.000000 0.000000 0.000000, axis 0 1 0, limit lower=-0.001 upper=0.001 effort=400 velocity=100
- added joint fsee_z: type prismatic, parent dummy_ee_sensor_link1, child end_effector, origin xyz=0.000000 0.000000 0.05000 rpy=0.000000 0.000000 0.000000, axis 0 0 1, limit lower=-0.001 upper=0.001 effort=400 velocity=100

Commit message: changed the way force sensor is simulated

File: robot_models/kuka_iiwa/03-multi_contact_validation/kuka_iiwa_base_sensor.urdf (robot description, URDF)
Before this commit: robot kuka_iiwa, 14 links, 13 joints
Links:
- removed link dummy_ee_sensor_link0
- removed link dummy_ee_sensor_link1
- removed link end_effector
- added link dummy_base_sensor_link3, mass 0.001
- added link dummy_base_sensor_link4, mass 0.001
- added link dummy_base_sensor_link5, mass 0.001
- link base_link: geometry collision box size=0.3 0.3 0.05; visual box size=0.3 0.3 0.05
- link link6: geometry collision sphere radius=0.035; visual mesh filename=../meshes/link6.obj scale=1 1 1
Joints:
- removed joint fsee_x
- removed joint fsee_y
- removed joint fsee_z
- added joint fsbase_tx: type revolute, parent dummy_base_sensor_link3, child dummy_base_sensor_link4, origin xyz=0.000000 0.000000 0.00000 rpy=0.000000 0.000000 0.000000, axis 1 0 0, limit lower=-0.001 upper=0.001 effort=400 velocity=100
- added joint fsbase_ty: type revolute, parent dummy_base_sensor_link4, child dummy_base_sensor_link5, origin xyz=0.000000 0.000000 0.00000 rpy=0.000000 0.000000 0.000000, axis 0 1 0, limit lower=-0.001 upper=0.001 effort=400 velocity=100
- added joint fsbase_tz: type revolute, parent dummy_base_sensor_link5, child base_link, origin xyz=0.000000 0.000000 0.00000 rpy=0.000000 0.000000 0.000000, axis 0 0 1, limit lower=-0.001 upper=0.001 effort=400 velocity=100
- joint fsbase_z: child base_link -> dummy_base_sensor_link3
