Commit message: implementation of current best guess on how to find Rc

File: 00-passivity_tests/kuka_iiwa.urdf (robot description, URDF)
Before this commit: robot kuka_iiwa, 8 links, 7 joints
Links:
- link link6: geometry collision sphere radius=0.04; visual mesh filename=../../../robot_models/kuka_iiwa/meshes/link6.obj scale=1 1 1
