Commit message: example passivity with square end effector

File: 04-passivity_demo_square_ee/iiwa7.urdf (robot description, URDF)
Before this commit: robot kuka_iiwa, 8 links, 7 joints
Links:
- removed link link0
- added link link7, mass 3.529; collision box size=0.08 0.08 0.08; visual box size=0.08 0.08 0.08
- link base_link: mass 4 -> 5
- link link1: mass 4 -> 3.4525; geometry visual mesh filename=../../../robot_models/kuka_iiwa/meshes/link0.obj scale=1 1 1
- link link2: mass 4 -> 3.4821; geometry visual mesh filename=../../../robot_models/kuka_iiwa/meshes/link1.obj scale=1 1 1
- link link3: mass 4 -> 4.05623; geometry visual mesh filename=../../../robot_models/kuka_iiwa/meshes/link2.obj scale=1 1 1
- link link4: mass 3 -> 3.4822; geometry visual mesh filename=../../../robot_models/kuka_iiwa/meshes/link3.obj scale=1 1 1
- link link5: mass 2 -> 2.1633; geometry visual mesh filename=../../../robot_models/kuka_iiwa/meshes/link4.obj scale=1 1 1
- link link6: mass 1 -> 2.3466; geometry visual mesh filename=../../../robot_models/kuka_iiwa/meshes/link5.obj scale=1 1 1
Joints:
- joint j0: child link0 -> link1; origin xyz=0.000000 0.000000 0.155767 rpy=0.000000 0.000000 0.000000 -> xyz=0 0 0.15 rpy=0 0 0
- joint j1: child link1 -> link2; origin xyz=0.000000 0.000000 0.182500 rpy=0.000000 0.000000 0.000000 -> xyz=0.000000 0.000000 0.19 rpy=0.000000 0.000000 0.000000; parent link0 -> link1
- joint j2: child link2 -> link3; origin xyz=0.000000 0.000000 0.185000 rpy=0.000000 0.000000 0.000000 -> xyz=0.000000 0.000000 0.21 rpy=0.000000 0.000000 0.000000; parent link1 -> link2
- joint j3: child link3 -> link4; origin xyz=0.000000 0.000000 0.217000 rpy=0.000000 0.000000 3.1415926535897 -> xyz=0.000000 0.000000 0.19 rpy=0.000000 0.000000 3.1415926535897; parent link2 -> link3
- joint j4: child link4 -> link5; origin xyz=0.000000 0.000000 0.186000 rpy=0.000000 0.000000 -3.1415926535897 -> xyz=0.000000 0.000000 0.21 rpy=0.000000 0.000000 -3.1415926535897; parent link3 -> link4
- joint j5: child link5 -> link6; origin xyz=0.000000 0.000000 0.217003 rpy=0.000000 0.000000 0.000000 -> xyz=0.000000 -0.06070 0.19 rpy=0.000000 0.000000 0.000000; parent link4 -> link5
- joint j6: child link6 -> link7; origin xyz=0.000000 0.000000 0.081000 rpy=0.000000 0.000000 0.000000 -> xyz=0.000000 0.06070 0.081000 rpy=0.000000 0.000000 0.000000; parent link5 -> link6
